File: Hardware/Electronics/Custom PCBs/Magnetic Angle Sensor Breakout v2/magn_angle_sensor_v2/magn_angle_sensor_v2.kicad_sch (KiCad schematic)
At the start: 6 parts, among them J1 USB_C_Receptacle_USB2.0_16P, SW1 SW_Push, SW2 SW_Push, U1 RP2040, U2 W25Q128JVS, U3 SN65HVD1050D

Commit message: V2 magnetic sensor work
Parts:
- removed J1: USB_C_Receptacle_USB2.0_16P, symbol Connector:USB_C_Receptacle_USB2.0_16P
- removed SW1, SW2: SW_Push, symbol Switch:SW_Push
- added 3.3V1: 3.3V, TestPoint:TestPoint_Pad_D1.0mm, symbol Connector:TestPoint
- added BOOT1: USB_BOOT, Button_Switch_SMD:SW_SPST_B3U-1000P, symbol Switch:SW_Push
- added C1, C12, C13, C14, C15, C16, C18, C21, C22, C6 (x2), C8, C9: 100n, Capacitor_SMD:C_0402_1005Metric, symbol Device:C
- added C11, C19, C20, C23, C24, C7: 1u, Capacitor_SMD:C_0402_1005Metric, symbol Device:C
- added C17: 1u/100V, Capacitor_SMD:C_0805_2012Metric, symbol Device:C
- added C2, C3: 22p, Capacitor_SMD:C_0402_1005Metric, symbol Device:C
- added C4, C5: 47p, Capacitor_SMD:C_0402_1005Metric, symbol Device:C
- added CR1: PESD1CAN_215, Package_TO_SOT_SMD:SOT-23, symbol symbols:PESD1CAN_215
- added D1: LED, LED_SMD:LED_0402_1005Metric, symbol Device:LED
- added H1, H2: MountingHole, MountingHole:MountingHole_3.2mm_M3_DIN965_Pad, symbol Mechanical:MountingHole
- added J1: JST PH 01x04, Connector_JST:JST_PH_S4B-PH-K_1x04_P2.00mm_Horizontal, symbol Connector_Generic:Conn_01x04
- added J2: USB C Receptacle, Connector_USB:USB_C_Receptacle_G-Switch_GT-USB-7010ASV, symbol Connector:USB_C_Receptacle_USB2.0
- added J3: 120TR, Connector_PinHeader_2.54mm:PinHeader_1x02_P2.54mm_Vertical, symbol Connector_Generic:Conn_01x02
- added R1, R7: 10k, Resistor_SMD:R_0402_1005Metric, symbol Device:R
- added R13: 120, Resistor_SMD:R_0402_1005Metric, symbol Device:R
- added R13: NC, Resistor_SMD:R_0402_1005Metric, symbol Device:R
- added R2: 1k, Resistor_SMD:R_0402_1005Metric, symbol Device:R
- added R3, R4: 5.1k, Resistor_SMD:R_0402_1005Metric, symbol Device:R
- added R5, R6: 27.4, Resistor_SMD:R_0402_1005Metric, symbol Device:R
- added R5: 1K, Resistor_SMD:R_0402_1005Metric, symbol Device:R
- added R6: 10K, Resistor_SMD:R_0402_1005Metric, symbol Device:R
- added RESET1: RESET, Button_Switch_SMD:SW_SPST_B3U-1000P, symbol Switch:SW_Push
- added SCL1: SCL, TestPoint:TestPoint_Pad_D1.0mm, symbol Connector:TestPoint
- added SDA1: SDA, TestPoint:TestPoint_Pad_D1.0mm, symbol Connector:TestPoint
- added TP2: GND, TestPoint:TestPoint_Pad_D1.0mm, symbol Connector:TestPoint
- added TP5: D0, TestPoint:TestPoint_Pad_D1.0mm, symbol Connector:TestPoint
- added TP6: D1, TestPoint:TestPoint_Pad_D1.0mm, symbol Connector:TestPoint
- added U1: MT6701-CT, Package_SO:SOP-8_3.9x4.9mm_P1.27mm, symbol symbols:MT6701-CT
- added U4: SE8650X2-HF, Package_TO_SOT_SMD:SOT-23, symbol Regulator_Linear:LF15_TO220
- added U6: XC6206P332MR, Package_TO_SOT_SMD:SOT-23, symbol Regulator_Linear:LF15_TO220
- added Y1: 12MHz/12pF/50Ω/20ppm, Crystal:Crystal_SMD_3225-4Pin_3.2x2.5mm, symbol Device:Crystal_GND24
- U2: LCSC (none) -> C97521
- renumbered U1 to U2, U3 to U5
Connections:
- net CAN_TX: now reaches U5.1 (TXD)
- net CAN_TX: now also U2.7 (GPIO5)
- net GND: now reaches U5.2 (GND)
- net GND: now also U2.19 (TESTEN), U2.4 (GND), U2.57 (GND), BOOT1.1, C1.2, C11.2, C12.1, C13.1, C14.1, C15.1, C16.1, C17.1, C18.1, C19.1, C2.1, C20.2, C21.1, C22.2, C23.2, C24.2, C3.1, C4.2, C5.2, C6.1, C6.2, C7.1, C8.1, C9.1, CR1.3, D1.1 (K), J1.4 (Pin_4), J2.A1 (GND), J2.A12 (GND), J2.B1 (GND), J2.B12 (GND), J2.S1 (SHIELD), R3.2, R4.2, RESET1.1, TP2.1, U1.4 (GND), U4.1 (GND), U6.1 (GND), Y1.2, Y1.4
- net +5V: now reaches U5.3 (VCC)
- net +5V: now also C19.2, C20.1, C21.2, C23.1, U4.2 (VO), U6.3 (VI)
- net CAN_RX: now reaches U5.4 (RXD)
- net CAN_RX: now also U2.6 (GPIO4)
- net at U5.5 (VREF): now also C22.1
- net CAN_L: now reaches U5.6 (CANL)
- net CAN_L: now also C5.1, CR1.2, J1.3 (Pin_3), R13.2
- net CAN_H: now reaches U5.7 (CANH)
- net CAN_H: now also C4.1, CR1.1, J1.2 (Pin_2), J3.2 (Pin_2)
- net at U5.8 (S): now also R13.1
- net QSPI_SS: now reaches U2.1 (~{CS})
- net QSPI_SS: now also U2.56 (QSPI_SS), R5.2, R6.1
- net QSPI_SD1: now reaches U2.2 (DO(IO1))
- net QSPI_SD1: now also U2.55 (QSPI_SD1)
- net QSPI_SD2: now reaches U2.3 (IO2)
- net QSPI_SD2: now also U2.54 (QSPI_SD2)
- net QSPI_SD0: now reaches U2.5 (DI(IO0))
- net QSPI_SD0: now also U2.53 (QSPI_SD0)
- net QSPI_SCK: now reaches U2.6 (CLK)
- net QSPI_SCK: now also U2.52 (QSPI_SCLK)
- net QSPI_SD3: now reaches U2.7 (IO3)
- net QSPI_SD3: now also U2.51 (QSPI_SD3)
- net +3.3V: now reaches U2.8 (VCC)
- net +3.3V: now also U2.1 (IOVDD), U2.10 (IOVDD), U2.22 (IOVDD), U2.33 (IOVDD), U2.42 (IOVDD), U2.43 (ADC_AVDD), U2.44 (VREG_IN), U2.48 (USB_VDD), U2.49 (IOVDD), 3.3V1.1, C1.1, C11.1, C12.2, C13.2, C14.2, C15.2, C16.2, C18.2, C24.1, C6.1, C9.2, R6.2, R7.1, U1.1 (VDD), U1.2 (MODE), U6.2 (VO)
- net LED: now reaches U2.16 (GPIO13)
- net LED: now also R1.2
- net at U2.2 (GPIO0): now also TP5.1
- net at U2.20 (XIN): now also C2.2, Y1.3
- net at U2.21 (XOUT): now also R2.2
- net +1V1: now reaches U2.23 (DVDD), U2.50 (DVDD)
- net +1V1: now also U2.45 (VREG_VOUT), C6.2, C7.2, C8.2
- net RUN: now reaches U2.26 (RUN)
- net RUN: now also R7.2, RESET1.2
- net at U2.3 (GPIO1): now also TP6.1
- net SDA: now reaches U2.4 (GPIO2)
- net SDA: now also SDA1.1, U1.6 (A/U/SDA/DO)
- net at U2.46 (USB_DM): now also R6.1
- net at U2.47 (USB_DP): now also R5.2
- net SCL: now reaches U2.5 (GPIO3)
- net SCL: now also SCL1.1, U1.7 (B/V/SCL/CLK)
- net CAN_S: now reaches U2.8 (GPIO6)
- net CAN_S: now also R13.2
- new net: J3.1 (Pin_1), R13.1
- new net: J2.A5 (CC1), R4.1
- new net: J2.B5 (CC2), R3.1
- new net: C3.2, R2.1, Y1.1
- new net: D1.2 (A), R1.1
- new net +24V: C17.2, J1.1 (Pin_1), U4.3 (VI)
- new net USB_D+: J2.A6 (D+), J2.B6 (D+), R5.1
- new net USB_D-: J2.A7 (D-), J2.B7 (D-), R6.2
- new net VBUS: J2.A4 (VBUS), J2.A9 (VBUS), J2.B4 (VBUS), J2.B9 (VBUS)
- new net ~{USB_BOOT}: BOOT1.2, R5.1
- no-connect marks 0 -> 29
Other:
- moved on the sheet: U2, U5

Commit message: Finish CAN Magnetic Angle Sensor v2
Parts:
- removed 3.3V1: 3.3V, TestPoint:TestPoint_Pad_D1.0mm, symbol Connector:TestPoint
- removed C1, C14, C21, C6 (x2): 100n, Capacitor_SMD:C_0402_1005Metric, symbol Device:C
- removed C17: 1u/100V, Capacitor_SMD:C_0805_2012Metric, symbol Device:C
- removed C2, C3: 22p, Capacitor_SMD:C_0402_1005Metric, symbol Device:C
- removed C20, C23, C24: 1u, Capacitor_SMD:C_0402_1005Metric, symbol Device:C
- removed C4, C5: 47p, Capacitor_SMD:C_0402_1005Metric, symbol Device:C
- removed R13: 120, Resistor_SMD:R_0402_1005Metric, symbol Device:R
- removed R13: NC, Resistor_SMD:R_0402_1005Metric, symbol Device:R
- removed R4: 5.1k, Resistor_SMD:R_0402_1005Metric, symbol Device:R
- removed R5, R6: 27.4, Resistor_SMD:R_0402_1005Metric, symbol Device:R
- removed R5: 1K, Resistor_SMD:R_0402_1005Metric, symbol Device:R
- removed R6: 10K, Resistor_SMD:R_0402_1005Metric, symbol Device:R
- removed SCL1: SCL, TestPoint:TestPoint_Pad_D1.0mm, symbol Connector:TestPoint
- removed SDA1: SDA, TestPoint:TestPoint_Pad_D1.0mm, symbol Connector:TestPoint
- removed U2: RP2040, Package_DFN_QFN:QFN-56-1EP_7x7mm_P0.4mm_EP3.2x3.2mm, symbol MCU_RaspberryPi:RP2040
- removed U4: SE8650X2-HF, Package_TO_SOT_SMD:SOT-23, symbol Regulator_Linear:LF15_TO220
- removed U5: SN65HVD1050D, Package_SO:SOIC-8_3.9x4.9mm_P1.27mm, symbol Interface_CAN_LIN:SN65HVD1050D
- removed U6: XC6206P332MR, Package_TO_SOT_SMD:SOT-23, symbol Regulator_Linear:LF15_TO220
- added C1 (x2), C2, C3, C4, C5, C6 (x2): 100n, Capacitor_SMD:C_0402_1005Metric, symbol Device:C
- added C10: 1u/100V, Capacitor_SMD:C_0805_2012Metric, symbol Device:C
- added C2, C3: 22p, Capacitor_SMD:C_0402_1005Metric, symbol Device:C
- added C4, C5: 47p, Capacitor_SMD:C_0402_1005Metric, symbol Device:C
- added R13: NC, Resistor_SMD:R_0402_1005Metric, symbol Device:R
- added R13: 120, Resistor_SMD:R_0402_1005Metric, symbol Device:R
- added R4: 5.1k, Resistor_SMD:R_0402_1005Metric, symbol Device:R
- added R4, R5: 27.4, Resistor_SMD:R_0402_1005Metric, symbol Device:R
- added R5: 1K, Resistor_SMD:R_0402_1005Metric, symbol Device:R
- added R6: 10K, Resistor_SMD:R_0402_1005Metric, symbol Device:R
- added TP1: D0, TestPoint:TestPoint_Pad_D1.0mm, symbol Connector:TestPoint
- added TP3: SCL, TestPoint:TestPoint_Pad_D1.0mm, symbol Connector:TestPoint
- added TP4: SDA, TestPoint:TestPoint_Pad_D1.0mm, symbol Connector:TestPoint
- added U1: SE8650X2-HF, Package_TO_SOT_SMD:SOT-23, symbol Regulator_Linear:LF15_TO220
- added U2: XC6206P332MR, Package_TO_SOT_SMD:SOT-23, symbol Regulator_Linear:LF15_TO220
- added U5: RP2040, Package_DFN_QFN:QFN-56-1EP_7x7mm_P0.4mm_EP3.2x3.2mm, symbol MCU_RaspberryPi:RP2040
- added U6: SN65HVD1050D, Package_SO:SOIC-8_3.9x4.9mm_P1.27mm, symbol Interface_CAN_LIN:SN65HVD1050D
- BOOT1: value USB_BOOT -> BOOT
- C12, C13, C15, C16, C18: value 100n -> 1u
- C19, C7: value 1u -> 100n
- TP2: value GND -> D1
- TP5: value D0 -> 3.3V
- TP6: value D1 -> GND
Connections:
- net +1V1: now also C15.2, C1.2, C2.2, U5.23 (DVDD), U5.45 (VREG_VOUT), U5.50 (DVDD); no longer C7.2, C8.2
- net +24V: now also C10.2, U1.3 (VI)
- net +3.3V: now also C13.1, C16.1, C7.2, C8.2, TP5.1, C1.1, C3.2, C4.2, C5.2, C6.1, C6.2, R6.2, U2.2 (VO), U5.1 (IOVDD), U5.10 (IOVDD), U5.22 (IOVDD), U5.33 (IOVDD), U5.42 (IOVDD), U5.43 (ADC_AVDD), U5.44 (VREG_IN), U5.48 (USB_VDD), U5.49 (IOVDD); no longer C11.1, C12.2, C13.2, C15.2, C16.2, C18.2
- net +5V: now also C11.1, C12.1, C18.2, U1.2 (VO), U2.3 (VI), U6.3 (VCC)
- net CAN_H: now also C4.1, U6.7 (CANH)
- net CAN_L: now also C5.1, R13.2, U6.6 (CANL)
- net CAN_RX: now also U5.6 (GPIO4), U6.4 (RXD)
- net CAN_S: now also R13.2, U5.8 (GPIO6)
- net CAN_TX: now also U5.7 (GPIO5), U6.1 (TXD)
- net GND: now also C12.2, C13.2, C16.2, TP6.1, C1.1, C1.2, C10.1, C2.1, C2.1, C3.1, C3.1, C4.1, C4.2, C5.1, C5.2, C6.1, C6.2, R4.2, U1.1 (GND), U2.1 (GND), U5.19 (TESTEN), U5.57 (GND), U6.2 (GND); no longer C12.1, C13.1, C16.1, TP2.1
- net LED: now also U5.16 (GPIO13)
- net QSPI_SCK: now also U5.52 (QSPI_SCLK)
- net QSPI_SD0: now also U5.53 (QSPI_SD0)
- net QSPI_SD1: now also U5.55 (QSPI_SD1)
- net QSPI_SD2: now also U5.54 (QSPI_SD2)
- net QSPI_SD3: now also U5.51 (QSPI_SD3)
- net QSPI_SS: now also R5.2, R6.1, U5.56 (QSPI_SS)
- net RUN: now also U5.26 (RUN)
- net SCL: now also TP3.1, U5.5 (GPIO3)
- net SDA: now also TP4.1, U5.4 (GPIO2)
- net USB_D+: now also R4.1
- net USB_D-: now also R5.2
- net ~{USB_BOOT}: now also R5.1
- net at J3.1 (Pin_1): now also R13.1
- net at C22.1: now also U6.5 (VREF)
- net at J2.A5 (CC1): now also R4.1
- net at R2.1, Y1.1: now also C3.2
- net at R2.2: now also U5.21 (XOUT)
- net at Y1.3: now also C2.2, U5.20 (XIN)
- new net: R13.1, U6.8 (S)
- new net: TP1.1, U5.2 (GPIO0)
- new net: R5.1, U5.46 (USB_DM)
- new net: TP2.1, U5.3 (GPIO1)
- new net: R4.2, U5.47 (USB_DP)
Other:
- moved on the sheet: H1, H2
