File: Hardware/Electronics/Custom PCBs/Toolhead Board/Toolhead Board.kicad_pcb (KiCad board)
At the start: 4 copper layers, 75 x 75 mm, 172 parts, among them J1 USB C Receptacle, J10 Conn_01x02, J11 Conn_01x02, J12 120TR, J2 Conn_02x08_Odd_Even, J3 Conn_02x08_Odd_Even, J4 Conn_02x08_Odd_Even, J5 Conn_02x04_Odd_Even, J6 Conn_02x04_Odd_Even, Q1 MMBT4403, Q2 MMBT4403, Q3 MMBT4403, SW1 BOOT, SW2 RESET, U1 LF15_TO220, U10 BMI270, U11 G20N06D52, U12 G20N06D52, U13 PCA9685BS, U2 LF15_TO220, U3 RP2040, U4 W25Q128JVS, U5 SN65HVD1050D, U6 TMC2209-LA, U7 HX711, U8 HX711, U9 HX711, Y1 12MHz/12pF/50Ω/20ppm

Commit message: Updated PCB
Parts:
- moved R1 108.1 mm to (86.6, 101.8), turned to -163 degrees
- moved JP1 101.3 mm to (83.4, 102.7), turned to 17 degrees
- moved R14 91.4 mm to (86.1, 100.3), turned to 17 degrees
- moved TP3 83.8 mm to (109.0, 64.0)
- moved C29 81.8 mm to (98.1, 69.0)
- moved C27 81.6 mm to (98.0, 65.5), turned to 180 degrees
- moved C28 81.6 mm to (98.1, 67.5)
- moved R13 74.7 mm to (108.1, 68.5), turned to 180 degrees
- moved R12 74.6 mm to (108.0, 66.5)
- moved C5 67.1 mm to (114.6, 78.0)
- moved C7 66.9 mm to (114.1, 81.0)
- moved C8 66.8 mm to (114.4, 84.0)
- moved C24 61.7 mm to (116.0, 74.0)
- moved C10 58.0 mm to (121.6, 82.5)
- moved C11 58.0 mm to (126.0, 70.0)
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Routing:
- net /CAN IO/CAN_H: track 8.16 -> 71.2 mm, vias 1 -> 2
- net /CAN IO/CAN_L: track 14.8 -> 74.0 mm
- net OB1: track 0.00 -> 37.9 mm, vias 0 -> 2
- net Net-(JP5-B): track 0.00 -> 25.5 mm
- net Net-(JP6-B): track 0.00 -> 19.8 mm
- net /Microcontroller/RUN: track 0.00 -> 16.4 mm
- net Net-(JP7-B): track 0.00 -> 15.8 mm
- net Net-(U12-G1): track 0.00 -> 15.2 mm
- net Net-(U6-DIAG): track 0.00 -> 14.5 mm, vias 0 -> 2
- net V_MOT: track 21.9 -> 36.5 mm
- net +5V: track 71.6 -> 58.6 mm
- net Net-(JP8-B): track 0.00 -> 11.2 mm
- net Net-(U13-LED3): track 0.00 -> 8.75 mm
- net Net-(U6-CPO): track 0.00 -> 7.51 mm
- net Net-(JP4-B): track 0.00 -> 7.32 mm, vias 0 -> 2
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