File: Hardware/Electronics/Custom PCBs/Toolhead Board Breakout/Toolhead Board Breakout.kicad_pcb (KiCad board)
At the start: 2 copper layers, 75 x 75 mm, 38 parts, among them J1 Conn_02x08_Odd_Even, J10 Conn_01x03, J11 Conn_01x03, J12 Conn_01x03, J13 Conn_01x02, J14 Conn_01x04, J15 Conn_01x02, J17 Conn_01x02, J18 Conn_01x02, J2 Conn_02x08_Odd_Even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

Commit message: Updated Breakout Board
Routing:
- net 5VA: track 67.6 -> 66.7 mm
Changed lines of the file:
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@@
 	)
 	(segment
-		(start 63.254999 45.125001)
-		(end 56.038947 52.341053)
+		(start 99.420042 63.900042)
+		(end 80.645001 45.125001)
+		(width 0.35)
+		(layer "F.Cu")
+		(net 19)
+	)
+	(segment
+		(start 101.368422 68.648423)
+		(end 99.420042 66.700043)
+		(width 0.35)
+		(layer "F.Cu")
+		(net 19)
+	)
+	(segment
+		(start 68.054999 45.125001)
+		(end 60.838947 52.341053)
+		(width 0.35)
+		(layer "F.Cu")
+		(net 19)
+	)
+	(segment
+		(start 101.55261 72.501239)
+		(end 101.55261 73.237208)
+		(width 0.35)
+		(layer "F.Cu")
+		(net 19)
+	)
+	(segment
+		(start 101.55261 73.237208)
+		(end 101.157205 73.632613)
+		(width 0.35)
+		(layer "F.Cu")
+		(net 19)
+	)
+	(segment
+		(start 80.645001 45.125001)
+		(end 68.054999 45.125001)
+		(width 0.35)
+		(layer "F.Cu")
+		(net 19)
+	)
+	(segment
+		(start 101.157205 73.632613)
+		(end 100.980428 73.632613)
+		(width 0.35)
+		(layer "F.Cu")
+		(net 19)
+	)
+	(segment
+		(start 101.443297 72.391926)
+		(end 101.55261 72.501239)
 		(width 0.35)
 		(layer "F.Cu")
@@
 	)
 	(segment
-		(start 99.420042 63.900042)
-		(end 80.645001 45.125001)
-		(width 0.35)
-		(layer "F.Cu")
-		(net 19)
-	)
-	(segment
-		(start 101.55261 72.501239)
-		(end 101.55261 73.237208)
-		(width 0.35)
-		(layer "F.Cu")
-		(net 19)
-	)
-	(segment
-		(start 101.368422 68.648423)
-		(end 99.420042 66.700043)
-		(width 0.35)
-		(layer "F.Cu")
-		(net 19)
-	)
-	(segment
-		(start 101.55261 73.237208)
-		(end 101.157205 73.632613)
-		(width 0.35)
-		(layer "F.Cu")
-		(net 19)
-	)
-	(segment
-		(start 56.038947 52.341053)
+		(start 60.838947 52.341053)
 		(end 51.702786 52.341053)
-		(width 0.35)
-		(layer "F.Cu")
-		(net 19)
-	)
-	(segment
-		(start 101.157205 73.632613)
-		(end 100.980428 73.632613)
-		(width 0.35)
-		(layer "F.Cu")
-		(net 19)
-	)
-	(segment
-		(start 80.645001 45.125001)
-		(end 63.254999 45.125001)
-		(width 0.35)
-		(layer "F.Cu")
-		(net 19)
-	)
-	(segment
-		(start 101.443297 72.391926)
-		(end 101.55261 72.501239)
 		(width 0.35)
 		(layer "F.Cu")
@@
 	)
 	(segment
-		(start 86.56 105.489999)
-		(end 87.68 104.369999)
-		(width 2.5)
-		(layer "F.Cu")
-		(net 32)
-	)
-	(segment
 		(start 94.555032 94.924215)
 		(end 91.780032 90.117775)
@@
 	)
 	(segment
-		(start 87.68 104.369999)
-		(end 87.68 100.024024)
+		(start 85.740001 105.489999)
+		(end 87.68 103.55)
+		(width 2.5)
+		(layer "F.Cu")
+		(net 32)
+	)
+	(segment
+		(start 84.5 105.489999)
+		(end 85.740001 105.489999)
 		(width 2.5)
 		(layer "F.Cu")
@@
 	)
 	(segment
-		(start 84.5 105.489999)
-		(end 86.56 105.489999)
-		(width 2.5)
-		(layer "F.Cu")
-		(net 32)
-	)
-	(segment
-		(start 87.68 100.024024)
-		(end 90.354809 97.349215)
-		(width 2.5)
-		(layer "F.Cu")
-		(net 32)
-	)
-	(segment
 		(start 99.046356 97.901152)
 		(end 97.442602 96.297398)
@@
 	)
 	(segment
+		(start 87.68 103.55)
+		(end 87.68 100.024024)
+		(width 2.5)
+		(layer "F.Cu")
+		(net 32)
+	)
+	(segment
 		(start 96.069419 94.924215)
 		(end 94.555032 94.924215)
@@
 	)
 	(segment
+		(start 87.68 100.024024)
+		(end 90.354809 97.349215)
+		(width 2.5)
+		(layer "F.Cu")
+		(net 32)
+	)
+	(segment
 		(start 87.579809 92.542775)
 		(end 90.354809 97.349215)
@@
 	)
 	(segment
-		(start 84.5 105.489999)
-		(end 86.56 105.489999)
-		(width 2.5)
-		(layer "B.Cu")
-		(net 32)
-	)
-	(segment
-		(start 86.56 105.489999)
-		(end 87.75 104.299999)
-		(width 2.5)
-		(layer "B.Cu")
-		(net 32)
-	)
-	(segment
-		(start 87.75 99.954024)
+		(start 87.69 100.014024)
 		(end 90.354809 97.349215)
+		(width 2.5)
+		(layer "B.Cu")
+		(net 32)
+	)
+	(segment
+		(start 85.800001 105.489999)
+		(end 87.69 103.6)
 		(width 2.5)
 		(layer "B.Cu")
@@
 	)
 	(segment
-		(start 87.75 104.299999)
-		(end 87.75 99.954024)
+		(start 84.5 105.489999)
+		(end 85.800001 105.489999)
 		(width 2.5)
 		(layer "B.Cu")
@@
 		(width 2.5)
 		(layer "B.Cu")
+		(net 32)
+	)
+	(segment
+		(start 87.69 103.6)
+		(end 87.69 100.014024)
+		(width 2.5)
+		(layer "B.Cu")

Commit message: Update PCB
Routing:
- net +24V: track 157.6 -> 158.5 mm
- net 24V_PWM3: track 41.7 -> 42.4 mm
Changed lines of the file:
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@@
+	)
+	(segment
+		(start 48.155108 57.98)
+		(end 72.484364 57.98)
+		(width 1.5)
+		(layer "B.Cu")
+		(net 11)
 	)
 	(segment
@@
 	)
 	(segment
+		(start 72.484364 57.98)
+		(end 73.801034 59.29667)
+		(width 1.5)
+		(layer "B.Cu")
+		(net 11)
+	)
+	(segment
 		(start 77.270739 58.366965)
 		(end 76.000739 60.56667)
@@
 		(start 68.5 78.81)
 		(end 68.5 80.012081)
-		(width 1.5)
-		(layer "B.Cu")
-		(net 11)
-	)
-	(segment
-		(start 73.630008 59.125644)
-		(end 73.801034 59.29667)
-		(width 1.5)
-		(layer "B.Cu")
-		(net 11)
-	)
-	(segment
-		(start 45.766059 60.369049)
-		(end 47.009464 59.125644)
 		(width 1.5)
 		(layer "B.Cu")
@@
 	)
 	(segment
-		(start 47.009464 59.125644)
-		(end 73.630008 59.125644)
+		(start 45.766059 60.369049)
+		(end 48.155108 57.98)
 		(width 1.5)
 		(layer "B.Cu")
@@
 	)
 	(segment
-		(start 71.83 58.68)
-		(end 69.923503 58.68)
-		(width 0.75)
-		(layer "F.Cu")
-		(net 12)
-	)
-	(segment
-		(start 69.793503 58.55)
-		(end 60.92 58.55)
+		(start 73.03 55.39)
+		(end 70.73 57.69)
+		(width 0.75)
+		(layer "F.Cu")
+		(net 12)
+	)
+	(segment
+		(start 70.73 57.69)
+		(end 61.78 57.69)
 		(width 0.75)
 		(layer "F.Cu")
@@
 	)
 	(segment
-		(start 60.92 58.55)
-		(end 56.75172 62.71828)
+		(start 76.309029 55.39)
+		(end 73.03 55.39)
 		(width 0.75)
 		(layer "F.Cu")
@@
 	)
 	(segment
+		(start 56.75172 62.71828)
+		(end 44.911008 62.71828)
+		(width 0.75)
+		(layer "F.Cu")
+		(net 12)
+	)
+	(segment
+		(start 61.78 57.69)
+		(end 56.75172 62.71828)
+		(width 0.75)
+		(layer "F.Cu")
+		(net 12)
+	)
+	(segment
 		(start 79.470443 59.636965)
 		(end 79.470443 58.551414)
@@
 	)
 	(segment
-		(start 73.646033 56.50671)
-		(end 73.646033 56.863967)
-		(width 0.75)
-		(layer "F.Cu")
-		(net 12)
-	)
-	(segment
-		(start 69.923503 58.68)
-		(end 69.793503 58.55)
-		(width 0.75)
-		(layer "F.Cu")
-		(net 12)
-	)
-	(segment
-		(start 73.646033 56.863967)
-		(end 71.83 58.68)
-		(width 0.75)
-		(layer "F.Cu")
-		(net 12)
-	)
-	(segment
-		(start 76.309029 55.39)
-		(end 74.762743 55.39)
-		(width 0.75)
-		(layer "F.Cu")
-		(net 12)
-	)
-	(segment
-		(start 56.75172 62.71828)
-		(end 44.911008 62.71828)
-		(width 0.75)
-		(layer "F.Cu")
-		(net 12)
-	)
-	(segment
-		(start 74.762743 55.39)
-		(end 73.646033 56.50671)
-		(width 0.75)
-		(layer "F.Cu")
-		(net 12)
-	)
-	(segment
-		(start 82.599852 64.37667)
-		(end 80.725878 66.250644)
-		(width 0.75)
-		(layer "F.Cu")
-		(net 13)
-	)
-	(segment
-		(start 66.330644 66.250644)
-		(end 63.78 63.7)
-		(width 0.75)
-		(layer "F.Cu")
-		(net 13)
-	)
-	(segment
-		(start 63.78 63.7)
+		(start 62.82 63.7)
 		(end 46.203166 63.7)
 		(width 0.75)
@@
 	)
 	(segment
-		(start 80.725878 66.250644)
-		(end 66.330644 66.250644)
+		(start 82.599852 64.37667)
+		(end 80.186522 66.79)
 		(width 0.75)
 		(layer "F.Cu")
@@
 	)
 	(segment
+		(start 80.186522 66.79)
+		(end 65.91 66.79)
+		(width 0.75)
+		(layer "F.Cu")
+		(net 13)
+	)
+	(segment
+		(start 65.91 66.79)
+		(end 62.82 63.7)
+		(width 0.75)
+		(layer "F.Cu")
+		(net 13)
+	)
+	(segment
 		(start 82.599852 64.37667)
 		(end 84.799557 65.64667)
@@
 	)
 	(segment
-		(start 71.89167 61.99167)
-		(end 69.4 59.5)
-		(width 0.75)
-		(layer "F.Cu")
-		(net 14)
-	)
-	(segment
-		(start 61.631702 59.5)
-		(end 58.675851 62.455851)
-		(width 0.75)
-		(layer "F.Cu")
-		(net 14)
-	)
-	(segment
-		(start 69.4 59.5)
-		(end 61.631702 59.5)
-		(width 0.75)
-		(layer "F.Cu")
-		(net 14)
-	)
-	(segment
 		(start 78.045443 61.99167)
-		(end 71.89167 61.99167)
+		(end 73.76167 61.99167)
+		(width 0.75)
+		(layer "F.Cu")
+		(net 14)
+	)
+	(segment
+		(start 73.76167 61.99167)
+		(end 70.46 58.69)
+		(width 0.75)
+		(layer "F.Cu")
+		(net 14)
+	)
+	(segment
+		(start 70.46 58.69)
+		(end 62.441702 58.69)
 		(width 0.75)
 		(layer "F.Cu")
@@
 		(layer "F.Cu")
 		(net 14)
+	)
+	(segment
+		(start 62.441702 58.69)
+		(end 58.675851 62.455851)
+		(width 0.75)
+		(layer "F.Cu")
+		(net 14)
